Commit message: Fix rover physics, rewrite teleop controller, expand office environment
- Fix wheel_diameter (0.45->0.75) and wheel_separation (1.16->1.7) to match
  actual URDF geometry — root cause of erratic movement
- Reduce max_wheel_torque from 5000 to 50 — was generating 80,000N on a 98kg
  robot causing flips/jitter
- Add max_wheel_acceleration limit for smoother wheel response
- Match base_link collision box to visual (1.5x1.0x0.6) — stops wall clipping
- Rewrite teleop with time-based acceleration ramps, smooth angular steering,
  speed-dependent turn scaling, and keyboard auto-repeat debounce
- Expand world from 20x13m to 30x25m with 5 office cabins, 3 staircases,
  5m corridor and 4m doorways (all >2x rover width)
- Add missing package.xml deps (gazebo_ros, rclpy, geometry_msgs, gazebo_msgs)
- Fix X11 auth (xhost +local:), GPU device check, and arg quoting in run script

Co-Authored-By: Claude Opus 4.6 <noreply@anthropic.com>

File: bocbot_ws/src/bocbot/urdf/bocbot.urdf (robot description, URDF)
Before this commit: robot bocbot, 15 links, 14 joints
Links:
- link base_link: geometry collision box size=1.5 1.0 0.6; visual box size=1.5 1.0 0.6

File: bocbot_ws/src/bocbot/urdf/bocbot.urdf.xacro (robot description, xacro)
@@ -21,5 +21,5 @@
     <collision name='collision'>
       <origin xyz="0 0 0" rpy=" 0 0 0"/>
-      <geometry><box size="1.2 0.8 0.4"/></geometry>
+      <geometry><box size="1.5 1.0 0.6"/></geometry>
     </collision>
     <visual name='chassis_visual'>
