Commit message: Update environment to Mega Office Complex (30x30) and refine hexapedal physics

File: bocbot_ws/src/bocbot/urdf/bocbot.urdf (robot description, URDF)
Before this commit: robot bocbot, 14 links, 13 joints
Links:
- link back_left_wheel: mass 2.0 -> 0.8; geometry collision cylinder length=0.05 radius=0.075; visual cylinder length=0.05 radius=0.075
- link back_right_wheel: mass 2.0 -> 0.8; geometry collision cylinder length=0.05 radius=0.075; visual cylinder length=0.05 radius=0.075
- link base_link: mass 15.0 -> 3.0; geometry collision box size=0.28 0.18 0.10; visual box size=0.30 0.20 0.12
- link camera: mass 0.1 -> 0.01; geometry visual box size=0.03 0.05 0.03
- link front_left_wheel: mass 2.0 -> 0.8; geometry collision cylinder length=0.05 radius=0.075; visual cylinder length=0.05 radius=0.075
- link front_right_wheel: mass 2.0 -> 0.8; geometry collision cylinder length=0.05 radius=0.075; visual cylinder length=0.05 radius=0.075
- link hokuyo: mass 1e-5 -> 0.01; geometry visual cylinder length=0.04 radius=0.03
- link left_bogie_link: mass 1.5 -> 0.5; geometry collision box size=0.20 0.02 0.05; visual box size=0.04 0.04 0.05
- link left_rocker_arm: mass 2.0 -> 0.5; geometry collision box size=0.30 0.02 0.05; visual box size=0.04 0.04 0.05
- link mid_left_wheel: mass 2.0 -> 0.8; geometry collision cylinder length=0.05 radius=0.075; visual cylinder length=0.05 radius=0.075
- link mid_right_wheel: mass 2.0 -> 0.8; geometry collision cylinder length=0.05 radius=0.075; visual cylinder length=0.05 radius=0.075
- link right_bogie_link: mass 1.5 -> 0.5; geometry collision box size=0.20 0.02 0.05; visual box size=0.04 0.04 0.05
- link right_rocker_arm: mass 2.0 -> 0.5; geometry collision box size=0.30 0.02 0.05; visual box size=0.04 0.04 0.05
Joints:
- joint back_left_wheel_joint: limit effort=10000 velocity=1000 -> effort=100 velocity=20; origin xyz=-0.2 0.05 -0.1 rpy=0 0 0 -> xyz=-0.1 0.06 -0.05 rpy=0 0 0
- joint back_right_wheel_joint: limit effort=10000 velocity=1000 -> effort=100 velocity=20; origin xyz=-0.2 -0.05 -0.1 rpy=0 0 0 -> xyz=-0.1 -0.06 -0.05 rpy=0 0 0
- joint camera_joint: axis 0 1 0 -> (none); origin xyz=0.175 0 0 rpy=0 0 0 -> xyz=0.15 0 0 rpy=0 0 0
- joint front_left_wheel_joint: limit effort=10000 velocity=1000 -> effort=100 velocity=20; origin xyz=0.1 0.05 -0.1 rpy=0 0 0 -> xyz=0.2 0.06 -0.1 rpy=0 0 0
- joint front_right_wheel_joint: limit effort=10000 velocity=1000 -> effort=100 velocity=20; origin xyz=0.1 -0.05 -0.1 rpy=0 0 0 -> xyz=0.2 -0.06 -0.1 rpy=0 0 0
- joint hokuyo_joint: axis 0 1 0 -> (none); origin xyz=0 0 0.1 rpy=0 0 0 -> xyz=0.1 0 0.06 rpy=0 0 0
- joint left_bogie_pivot: limit lower=-0.78 upper=0.78 effort=500 velocity=100 -> effort=500 velocity=10; origin xyz=-0.2 0.0 0 rpy=0 0 0 -> xyz=-0.1 0.0 -0.05 rpy=0 0 0; type revolute -> continuous
- joint left_differential_axle: limit lower=-0.78 upper=0.78 effort=1000 velocity=100 -> effort=1000 velocity=10; origin xyz=0.0 0.15 0 rpy=0 0 0 -> xyz=0.0 0.13 0 rpy=0 0 0; type revolute -> continuous
- joint mid_left_wheel_joint: limit effort=10000 velocity=1000 -> effort=100 velocity=20; origin xyz=0.0 0.05 -0.1 rpy=0 0 0 -> xyz=0.1 0.06 -0.05 rpy=0 0 0
- joint mid_right_wheel_joint: limit effort=10000 velocity=1000 -> effort=100 velocity=20; origin xyz=0.0 -0.05 -0.1 rpy=0 0 0 -> xyz=0.1 -0.06 -0.05 rpy=0 0 0
- joint right_bogie_pivot: limit lower=-0.78 upper=0.78 effort=500 velocity=100 -> effort=500 velocity=10; origin xyz=-0.2 0.0 0 rpy=0 0 0 -> xyz=-0.1 0.0 -0.05 rpy=0 0 0; type revolute -> continuous
- joint right_differential_axle: limit lower=-0.78 upper=0.78 effort=1000 velocity=100 -> effort=1000 velocity=10; origin xyz=0.0 -0.15 0 rpy=0 0 0 -> xyz=0.0 -0.13 0 rpy=0 0 0; type revolute -> continuous
- joint robot_footprint_joint: origin xyz=0 0 0 rpy=0 0 0 -> xyz=0 0 0.15 rpy=0 0 0

File: bocbot_ws/src/bocbot/urdf/bocbot.urdf.xacro (robot description, xacro)
@@ -4,22 +4,23 @@
   <!-- Base footprint -->
   <link name="robot_footprint"></link>
+  <!-- Ground contact anchor. Start close to ground -->
   <joint name="robot_footprint_joint" type="fixed">
-    <origin xyz="0 0 0" rpy="0 0 0" />
+    <origin xyz="0 0 0.15" rpy="0 0 0" />
     <parent link="robot_footprint"/>
     <child link="base_link" />
   </joint>
-  <!-- Main Chassis (Green/White Box from images) -->
+  <!-- Main Chassis -->
   <link name='base_link'>
-    <pose>0 0 0.2 0 0 0</pose>
-    <inertial>
-      <mass value="15.0"/>
+    <inertial>
+      <!-- Reduced mass significantly to stop violent collision resolving -->
+      <mass value="3.0"/>
       <origin xyz="0 0 0" rpy=" 0 0 0"/>
-      <inertia ixx="0.1" ixy="0" ixz="0" iyy="0.1" iyz="0" izz="0.1" />
+      <inertia ixx="0.05" ixy="0" ixz="0" iyy="0.05" iyz="0" izz="0.05" />
     </inertial>
     <collision name='collision'>
       <origin xyz="0 0 0" rpy=" 0 0 0"/>
+      <!-- Made collision box slightly smaller than visual to prevent snagging -->
       <geometry>
-        <!-- Polyhedral shape approximated as a box for now -->
-        <box size="0.35 0.25 0.15"/>
+        <box size="0.28 0.18 0.10"/>
       </geometry>
     </collision>
@@ -27,17 +28,16 @@
       <origin xyz="0 0 0" rpy=" 0 0 0"/>
       <geometry>
-        <box size="0.35 0.25 0.15"/>
+        <box size="0.30 0.20 0.12"/>
       </geometry>
     </visual>
   </link>
   <gazebo reference="base_link">
-    <!-- Using Green to match the first two images -->
     <material>Gazebo/Green</material>
   </gazebo>
-  <!-- Sensors attached to base_link -->
+  <!-- Camera -->
   <link name="camera">
     <inertial>
-      <mass value="0.1"/>
-      <origin xyz="0.0 0.0 0.0" rpy=" 0 0 0"/>
+      <mass value="0.01"/>
+      <origin xyz="0 0 0" rpy=" 0 0 0"/>
       <inertia ixx="1e-6" ixy="0" ixz="0" iyy="1e-6" iyz="0" izz="1e-6" />
     </inertial>
@@ -45,17 +45,13 @@
       <origin xyz="0 0 0" rpy="0 0 0" />
       <geometry>
-        <box size="0.05 0.05 0.05"/>
+        <box size="0.03 0.05 0.03"/>
       </geometry>
     </visual>
-    <collision name="camera_colision">
-      <origin xyz="0 0 0" rpy="0 0 0" />
-      <geometry>
-        <box size="0.05 0.05 0.05"/>
-      </geometry>
-    </collision>
-  </link>
+    <!-- Removed camera collision entirely to stop internal intersection jitter -->
+  </link>
+  <!-- Hokuyo -->
   <link name="hokuyo">
     <inertial>
-      <mass value="1e-5"/>
+      <mass value="0.01"/>
       <origin xyz="0 0 0" rpy=" 0 0 0"/>
       <inertia ixx="1e-6" ixy="0" ixz="0" iyy="1e-6" iyz="0" izz="1e-6" />
@@ -64,34 +60,21 @@
       <origin xyz="0 0 0" rpy="0 0 0" />
       <geometry>
-        <box size="0.05 0.05 0.05"/>
+        <cylinder radius="0.03" length="0.04"/>
       </geometry>
     </visual>
-    <collision name="hokuyo_colision">
-      <origin xyz="0 0 0" rpy="0 0 0" />
-      <geometry>
-        <box size="0.1 0.1 0.1"/>
-      </geometry>
-    </collision>
+    <!-- Removed hokuyo collision entirely to stop internal intersection jitter -->
   </link>
   <joint type="fixed" name="camera_joint">
-    <!-- Centered in the front of the green hull -->
-    <origin xyz="0.175 0 0" rpy="0 0 0"/>
+    <origin xyz="0.15 0 0" rpy="0 0 0"/>
     <child link="camera"/>
     <parent link="base_link"/>
-    <axis xyz="0 1 0" rpy="0 0 0"/>
   </joint>
   <joint type="fixed" name="hokuyo_joint">
-    <!-- Mounted on top of the green hull -->
-    <origin xyz="0 0 0.1" rpy="0 0 0"/>
+    <origin xyz="0.1 0 0.06" rpy="0 0 0"/>
     <child link="hokuyo"/>
     <parent link="base_link"/>
-    <axis xyz="0 1 0" rpy="0 0 0"/>
-  </joint>
-  <gazebo reference="camera">
-    <material>Gazebo/Red</material>
-  </gazebo>
-  <gazebo reference="hokuyo">
-    <material>Gazebo/Black</material>
-  </gazebo>
+  </joint>
+  <gazebo reference="camera"><material>Gazebo/Black</material></gazebo>
+  <gazebo reference="hokuyo"><material>Gazebo/Black</material></gazebo>
   <!-- =============================== -->
   <!-- LEFT SIDE ROCKER-BOGIE ASSEMBLY -->
@@ -100,181 +83,166 @@
   <link name="left_rocker_arm">
     <inertial>
-      <mass value="2.0"/>
+      <!-- Ensure arm mass is much lower than base -->
+      <mass value="0.5"/>
       <origin xyz="0 0 0" rpy="0 0 0"/>
-      <inertia ixx="0.05" ixy="0" ixz="0" iyy="0.05" iyz="0" izz="0.05" />
-    </inertial>
-    <visual>
-      <origin xyz="-0.05 0.05 -0.05" rpy="0 0 0"/>
-      <geometry>
-        <box size="0.3 0.05 0.05"/>
-      </geometry>
-    </visual>
-    <collision>
-      <origin xyz="-0.05 0.05 -0.05" rpy="0 0 0"/>
-      <geometry>
-        <box size="0.3 0.05 0.05"/>
-      </geometry>
-    </collision>
-  </link>
-  <gazebo reference="left_rocker_arm">
-    <material>Gazebo/DarkGrey</material>
-  </gazebo>
-  <!-- Left Rocker to Chassis Joint (Pitch Revolute) -->
-  <joint name="left_differential_axle" type="revolute">
-    <origin xyz="0.0 0.15 0" rpy="0 0 0"/>
+      <inertia ixx="0.005" ixy="0" ixz="0" iyy="0.005" iyz="0" izz="0.005" />
+    </inertial>
+    <visual>
+      <origin xyz="0.05 0 0" rpy="0 0 0"/>
+      <geometry><box size="0.34 0.04 0.04"/></geometry>
+    </visual>
+    <visual>
+      <origin xyz="0.2 0 -0.05" rpy="0 0 0"/>
+      <geometry><box size="0.04 0.04 0.10"/></geometry>
+    </visual>
+    <visual>
+      <origin xyz="-0.1 0 -0.025" rpy="0 0 0"/>
+      <geometry><box size="0.04 0.04 0.05"/></geometry>
+    </visual>
+    <collision>
+      <origin xyz="0.05 0 -0.025" rpy="0 0 0"/>
+      <!-- Thinned the collision box -->
+      <geometry><box size="0.30 0.02 0.05"/></geometry>
+    </collision>
+  </link>
+  <gazebo reference="left_rocker_arm"><material>Gazebo/DarkGrey</material></gazebo>
+  <!-- To fix "jumping", we switch this from revolute to continuous for Gazebo solver stability -->
+  <joint name="left_differential_axle" type="continuous">
+    <origin xyz="0.0 0.13 0" rpy="0 0 0"/>
     <parent link="base_link"/>
     <child link="left_rocker_arm"/>
     <axis xyz="0 1 0"/>
-    <limit lower="-0.78" upper="0.78" effort="1000" velocity="100"/>
+    <limit effort="1000" velocity="10"/>
+    <!-- Provide reasonable friction to prevent floppy legs -->
     <dynamics damping="5.0" friction="5.0"/>
   </joint>
-  <!-- Left Front Wheel Module -->
+  <!-- Left Front Wheel -->
   <link name="front_left_wheel">
     <inertial>
-      <mass value="2.0"/>
-      <origin xyz="0 0 0" rpy="1.5707 0 0"/>
-      <inertia ixx="0.01" ixy="0" ixz="0" iyy="0.01" iyz="0" izz="0.01" />
-    </inertial>
-    <visual>
-      <origin xyz="0 0 0" rpy="1.5707 0 0"/>
-      <geometry>
-        <cylinder length="0.06" radius="0.075"/>
-      </geometry>
-    </visual>
-    <collision>
-      <origin xyz="0 0 0" rpy="1.5707 0 0"/>
-      <geometry>
-        <cylinder length="0.06" radius="0.075"/>
-      </geometry>
-      <surface>
-        <friction>
-          <ode>
-            <mu>1.0</mu>
-            <mu2>1.0</mu2>
-          </ode>
-        </friction>
-      </surface>
+      <mass value="0.8"/>
+      <origin xyz="0 0 0" rpy="1.5707 0 0"/>
+      <!-- Using exactly calculated cylinder inertia: 1/12m(3r^2+h^2), 1/2mr^2 -->
+      <inertia ixx="0.0013" ixy="0" ixz="0" iyy="0.0013" iyz="0" izz="0.0022" />
+    </inertial>
+    <visual>
+      <origin xyz="0 0 0" rpy="1.5707 0 0"/>
+      <geometry><cylinder length="0.05" radius="0.075"/></geometry>
+    </visual>
+    <collision>
+      <origin xyz="0 0 0" rpy="1.5707 0 0"/>
+      <geometry><cylinder length="0.05" radius="0.075"/></geometry>
     </collision>
   </link>
   <gazebo reference="front_left_wheel">
     <material>Gazebo/Grey</material>
+    <!-- Physics engine traction tags -->
+    <mu1>1.0</mu1>
+    <mu2>1.0</mu2>
+    <kp>1000000.0</kp>
+    <kd>100.0</kd>
   </gazebo>
   <joint name="front_left_wheel_joint" type="continuous">
-    <origin xyz="0.1 0.05 -0.1" rpy="0 0 0"/>
+    <origin xyz="0.2 0.06 -0.1" rpy="0 0 0"/>
     <parent link="left_rocker_arm"/>
     <child link="front_left_wheel"/>
     <axis xyz="0 1 0"/>
-    <limit effort="10000" velocity="1000"/>
-    <dynamics damping="1.0" friction="1.0"/>
-  </joint>
-  <!-- Left Bogie Link (Trailing) -->
+    <limit effort="100" velocity="20"/>
+    <dynamics damping="0.1" friction="0.1"/>
+  </joint>
+  <!-- Left Bogie Link -->
   <link name="left_bogie_link">
     <inertial>
-      <mass value="1.5"/>
-      <origin xyz="-0.1 0.05 -0.05" rpy="0 0 0"/>
-      <inertia ixx="0.03" ixy="0" ixz="0" iyy="0.03" iyz="0" izz="0.03" />
-    </inertial>
-    <visual>
-      <origin xyz="-0.1 0.05 -0.05" rpy="0 0 0"/>
-      <geometry>
-        <box size="0.25 0.04 0.04"/>
-      </geometry>
-    </visual>
-    <collision>
-      <origin xyz="-0.1 0.05 -0.05" rpy="0 0 0"/>
-      <geometry>
-        <box size="0.25 0.04 0.04"/>
-      </geometry>
-    </collision>
-  </link>
-  <gazebo reference="left_bogie_link">
-    <material>Gazebo/DarkGrey</material>
-  </gazebo>
-  <!-- Left Rocker to Bogie Joint (Passive Pitch) -->
-  <joint name="left_bogie_pivot" type="revolute">
-    <origin xyz="-0.2 0.0 0" rpy="0 0 0"/>
+      <mass value="0.5"/>
+      <origin xyz="0 0 0" rpy="0 0 0"/>
+      <inertia ixx="0.005" ixy="0" ixz="0" iyy="0.005" iyz="0" izz="0.005" />
+    </inertial>
+    <visual>
+      <origin xyz="0 0 0" rpy="0 0 0"/>
+      <geometry><box size="0.24 0.04 0.04"/></geometry>
+    </visual>
+    <visual>
+      <origin xyz="0.1 0 -0.025" rpy="0 0 0"/>
+      <geometry><box size="0.04 0.04 0.05"/></geometry>
+    </visual>
+    <visual>
+      <origin xyz="-0.1 0 -0.025" rpy="0 0 0"/>
+      <geometry><box size="0.04 0.04 0.05"/></geometry>
+    </visual>
+    <collision>
+      <origin xyz="0 0 -0.025" rpy="0 0 0"/>
+      <geometry><box size="0.20 0.02 0.05"/></geometry>
+    </collision>
+  </link>
+  <gazebo reference="left_bogie_link"><material>Gazebo/DarkGrey</material></gazebo>
+  <!-- Also changed to continuous for stability -->
+  <joint name="left_bogie_pivot" type="continuous">
+    <origin xyz="-0.1 0.0 -0.05" rpy="0 0 0"/>
     <parent link="left_rocker_arm"/>
     <child link="left_bogie_link"/>
     <axis xyz="0 1 0"/>
-    <limit lower="-0.78" upper="0.78" effort="500" velocity="100"/>
-    <dynamics damping="2.0" friction="2.0"/>
-  </joint>
-  <!-- Left Middle Wheel Module -->
+    <limit effort="500" velocity="10"/>
+    <dynamics damping="2.0" friction="1.0"/>
+  </joint>
+  <!-- Left Middle Wheel -->
   <link name="mid_left_wheel">
     <inertial>
-      <mass value="2.0"/>
-      <origin xyz="0 0 0" rpy="1.5707 0 0"/>
-      <inertia ixx="0.01" ixy="0" ixz="0" iyy="0.01" iyz="0" izz="0.01" />
-    </inertial>
-    <visual>
-      <origin xyz="0 0 0" rpy="1.5707 0 0"/>
-      <geometry>
-        <cylinder length="0.06" radius="0.075"/>
-      </geometry>
-    </visual>
-    <collision>
-      <origin xyz="0 0 0" rpy="1.5707 0 0"/>
-      <geometry>
-        <cylinder length="0.06" radius="0.075"/>
-      </geometry>
-      <surface>
-        <friction>
-          <ode>
-            <mu>1.0</mu>
-            <mu2>1.0</mu2>
-          </ode>
-        </friction>
-      </surface>
+      <mass value="0.8"/>
+      <origin xyz="0 0 0" rpy="1.5707 0 0"/>
+      <inertia ixx="0.0013" ixy="0" ixz="0" iyy="0.0013" iyz="0" izz="0.0022" />
+    </inertial>
+    <visual>
+      <origin xyz="0 0 0" rpy="1.5707 0 0"/>
+      <geometry><cylinder length="0.05" radius="0.075"/></geometry>
+    </visual>
+    <collision>
+      <origin xyz="0 0 0" rpy="1.5707 0 0"/>
+      <geometry><cylinder length="0.05" radius="0.075"/></geometry>
     </collision>
   </link>
   <gazebo reference="mid_left_wheel">
     <material>Gazebo/Grey</material>
+    <mu1>1.0</mu1>
+    <mu2>1.0</mu2>
+    <kp>1000000.0</kp>
+    <kd>100.0</kd>
   </gazebo>
   <joint name="mid_left_wheel_joint" type="continuous">
-    <origin xyz="0.0 0.05 -0.1" rpy="0 0 0"/>
+    <origin xyz="0.1 0.06 -0.05" rpy="0 0 0"/>
     <parent link="left_bogie_link"/>
     <child link="mid_left_wheel"/>
     <axis xyz="0 1 0"/>
-    <limit effort="10000" velocity="1000"/>
-    <dynamics damping="1.0" friction="1.0"/>
-  </joint>
-  <!-- Left Rear Wheel Module -->
+    <limit effort="100" velocity="20"/>
+    <dynamics damping="0.1" friction="0.1"/>
+  </joint>
+  <!-- Left Rear Wheel -->
   <link name="back_left_wheel">
     <inertial>
-      <mass value="2.0"/>
-      <origin xyz="0 0 0" rpy="1.5707 0 0"/>
-      <inertia ixx="0.01" ixy="0" ixz="0" iyy="0.01" iyz="0" izz="0.01" />
-    </inertial>
-    <visual>
-      <origin xyz="0 0 0" rpy="1.5707 0 0"/>
-      <geometry>
-        <cylinder length="0.06" radius="0.075"/>
-      </geometry>
-    </visual>
-    <collision>
-      <origin xyz="0 0 0" rpy="1.5707 0 0"/>
-      <geometry>
-        <cylinder length="0.06" radius="0.075"/>
-      </geometry>
-      <surface>
-        <friction>
-          <ode>
-            <mu>1.0</mu>
-            <mu2>1.0</mu2>
-          </ode>
-        </friction>
-      </surface>
+      <mass value="0.8"/>
+      <origin xyz="0 0 0" rpy="1.5707 0 0"/>
+      <inertia ixx="0.0013" ixy="0" ixz="0" iyy="0.0013" iyz="0" izz="0.0022" />
+    </inertial>
+    <visual>
+      <origin xyz="0 0 0" rpy="1.5707 0 0"/>
+      <geometry><cylinder length="0.05" radius="0.075"/></geometry>
+    </visual>
+    <collision>
+      <origin xyz="0 0 0" rpy="1.5707 0 0"/>
+      <geometry><cylinder length="0.05" radius="0.075"/></geometry>
     </collision>
   </link>
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
Commit message: Harden bocbot simulation controls and physics

File: bocbot_ws/src/bocbot/urdf/bocbot.urdf (robot description, URDF)
Before this commit: robot bocbot, 15 links, 14 joints
Links:
- link left_bogie_link: geometry collision box size=1.2 0.2 0.2; visual box size=1.2 0.2 0.2
- link left_rocker_arm: geometry collision box size=1.7 0.2 0.2; visual box size=1.7 0.2 0.2
- link right_bogie_link: geometry collision box size=1.2 0.2 0.2; visual box size=1.2 0.2 0.2
- link right_rocker_arm: geometry collision box size=1.7 0.2 0.2; visual box size=1.7 0.2 0.2

File: bocbot_ws/src/bocbot/urdf/bocbot.urdf.xacro (robot description, xacro)
@@ -70,4 +70,5 @@
       <mu1>1.5</mu1>
       <mu2>0.02</mu2> <!-- Almost zero lateral friction to allow easy pivot -->
+      <fdir1>1 0 0</fdir1> <!-- Align primary friction with wheel roll direction -->
       <kp>1000000.0</kp>
       <kd>100.0</kd>
@@ -91,4 +92,5 @@
     </inertial>
     <visual><origin xyz="0.25 0 0"/><geometry><box size="1.7 0.2 0.2"/></geometry></visual>
+    <collision><origin xyz="0.25 0 0"/><geometry><box size="1.7 0.2 0.2"/></geometry></collision>
   </link>
   <gazebo reference="left_rocker_arm"><material>Gazebo/DarkGrey</material></gazebo>
@@ -110,4 +112,5 @@
     </inertial>
     <visual><origin xyz="0 0 0"/><geometry><box size="1.2 0.2 0.2"/></geometry></visual>
+    <collision><origin xyz="0 0 0"/><geometry><box size="1.2 0.2 0.2"/></geometry></collision>
   </link>
   <gazebo reference="left_bogie_link"><material>Gazebo/DarkGrey</material></gazebo>
@@ -132,4 +135,5 @@
     </inertial>
     <visual><origin xyz="0.25 0 0"/><geometry><box size="1.7 0.2 0.2"/></geometry></visual>
+    <collision><origin xyz="0.25 0 0"/><geometry><box size="1.7 0.2 0.2"/></geometry></collision>
   </link>
   <gazebo reference="right_rocker_arm"><material>Gazebo/DarkGrey</material></gazebo>
@@ -151,4 +155,5 @@
     </inertial>
     <visual><origin xyz="0 0 0"/><geometry><box size="1.2 0.2 0.2"/></geometry></visual>
+    <collision><origin xyz="0 0 0"/><geometry><box size="1.2 0.2 0.2"/></geometry></collision>
   </link>
   <gazebo reference="right_bogie_link"><material>Gazebo/DarkGrey</material></gazebo>
